Commit message: change color

File: src/champ/champ_description/urdf/champ.urdf.xacro (robot description, xacro)
@@ -2,5 +2,5 @@
 <robot name="champ" xmlns:xacro="http://ros.org/wiki/xacro">
     <xacro:include filename="$(find champ_description)/urdf/properties.urdf.xacro" />
-    <material name="black"><color rgba="1.0 1.0 1.0 1.0" /></material>
+    <material name="black"><color rgba="0.0 0.0 1.0 1.0" /></material>
     <link name="base_link">
         <collision>

File: src/champ/champ_description/urdf/leg.urdf.xacro (robot description, xacro)
@@ -41,5 +41,5 @@
         </link>
         <gazebo reference="${leg}_hip_link">
-            <material>Gazebo/FlatBlack</material>
+            <material>Gazebo/Blue</material>
         </gazebo>
         <link name="${leg}_upper_leg_link">
@@ -66,5 +66,5 @@
         </link>
         <gazebo reference="${leg}_upper_leg_link">
-            <material>Gazebo/FlatBlack</material>
+            <material>Gazebo/Blue</material>
         </gazebo>
         <link name="${leg}_lower_leg_link">
@@ -96,5 +96,5 @@
             <mu2>0.8</mu2>
             <minDepth>0.05</minDepth>
-            <material>Gazebo/FlatBlack</material>
+            <material>Gazebo/Blue</material>
         </gazebo>
         <link name="${leg}_foot_link" />
