Commit message: backup before testing

File: src/champ/champ_description/urdf/accessories.urdf.xacro (robot description, xacro)
@@ -2,8 +2,8 @@
 <robot xmlns:xacro="http://ros.org/wiki/xacro">
     <xacro:macro name="accessories" params="base_name base_length base_height  " >
-        <xacro:include filename="$(find champ_description)/urdf/hokuyo_utm30lx.urdf.xacro" />
+        <xacro:include filename="$(find champ_description)/urdf/lidar_utm30lx.urdf.xacro" />
         <xacro:include filename="$(find champ_description)/urdf/asus_camera.urdf.xacro" />
-        <xacro:hokuyo_utm30lx
-            name="hokuyo"
+        <xacro:lidar_utm30lx
+            name="lidar"
             parent="${base_name}"
             ros_topic="scan"
@@ -13,5 +13,5 @@
             max_angle="130" >
             <origin xyz="0.0 0.0 ${base_height / 2 + 0.04}" rpy="0 0 0"/>
-        </xacro:hokuyo_utm30lx>
+        </xacro:lidar_utm30lx>
         <xacro:asus_camera
             parent="${base_name}"

File: src/champ/champ_description/urdf/champ.urdf (robot description, URDF)
Before this commit: robot champ, 29 links, 28 joints
Links:
- removed link hokuyo_frame
- added link lidar_frame, mass 0.270; collision box size=0.058 0.058 0.087; visual mesh filename=file:///home/Alexander.Karavaev/champ_ws/install/champ_desc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
Joints:
- removed joint hokuyo_joint
- added joint lidar_joint: type fixed, parent base_link, child lidar_frame, origin xyz=0.0 0.0 0.10500000000000001 rpy=0 0 0

File: src/champ/champ_description/urdf/lidar_utm30lx.urdf.xacro (robot description, xacro)
@@ -2,5 +2,5 @@
 <robot xmlns:xacro="http://www.ros.org/wiki/xacro">
     <xacro:property name="M_PI" value="3.1415926535897931" />
-    <xacro:macro name="hokuyo_utm30lx_model" params="name parent *origin">
+    <xacro:macro name="lidar_utm30lx_model" params="name parent *origin">
       <joint name="${name}_joint" type="fixed">
         <xacro:insert_block name="origin" />
@@ -17,5 +17,5 @@
           <origin xyz="0 0 0" rpy="0 0 0" />
           <geometry>
-          <mesh filename="file://$(find champ_description)/meshes/hokuyo_utm_30lx$(optenv TEST_SELF_FILTER).dae"/>
+          <mesh filename="file://$(find champ_description)/meshes/lidar_utm_30lx$(optenv TEST_SELF_FILTER).dae"/>
         </geometry>
         </visual>
@@ -24,13 +24,13 @@
           <geometry>
           <box size="0.058 0.058 0.087" />
-          <!--<mesh filename="package://hector_sensors_description/meshes/hokuyo_utm30lx/hokuyo_utm_30lx.stl"/>-->
+          <!--<mesh filename="package://hector_sensors_description/meshes/lidar_utm30lx/lidar_utm_30lx.stl"/>-->
         </geometry>
         </collision>
       </link>
     </xacro:macro>
-    <xacro:macro name="hokuyo_utm30lx" params="name parent *origin ros_topic update_rate ray_count min_angle max_angle">
-      <xacro:hokuyo_utm30lx_model name="${name}" parent="${parent}">
+    <xacro:macro name="lidar_utm30lx" params="name parent *origin ros_topic update_rate ray_count min_angle max_angle">
+      <xacro:lidar_utm30lx_model name="${name}" parent="${parent}">
         <xacro:insert_block name="origin" />
-      </xacro:hokuyo_utm30lx_model>
+      </xacro:lidar_utm30lx_model>
       <gazebo reference="${name}_frame">
         <sensor type="ray" name="${name}">
@@ -70,8 +70,8 @@
       </gazebo>
     </xacro:macro>
-    <xacro:macro name="hokuyo_utm30lx_gpu" params="name parent *origin ros_topic update_rate ray_count min_angle max_angle">
-      <xacro:hokuyo_utm30lx_model name="${name}" parent="${parent}">
+    <xacro:macro name="lidar_utm30lx_gpu" params="name parent *origin ros_topic update_rate ray_count min_angle max_angle">
+      <xacro:lidar_utm30lx_model name="${name}" parent="${parent}">
         <xacro:insert_block name="origin" />
-      </xacro:hokuyo_utm30lx_model>
+      </xacro:lidar_utm30lx_model>
       <gazebo reference="${name}_frame">
         <sensor type="gpu_ray" name="${name}">
